Commit message: minor numerical modifications

File: robot.urdf (robot description, URDF)
Before this commit: robot onshape, 4 links, 3 joints
Joints:
- joint cyl_z: type revolute -> prismatic

Commit message: more minor numerical modifications (personal preference)

File: robot.urdf (robot description, URDF)
Before this commit: robot onshape, 4 links, 3 joints
Joints:
- joint cyl_z: origin xyz=0 -0.063500000000000000888 -0.076200000000000017719 rpy=1.570796326794896558 -0 0 -> xyz=0 -0.0635 -0.0762 rpy=1.570796326794896558 -0 0

Commit message: convert negative zero to regular zero

File: robot.urdf (robot description, URDF)
Before this commit: robot onshape, 4 links, 3 joints
Joints:
- joint cyl_z: origin xyz=0 -0.0635 -0.0762 rpy=1.570796326794896558 -0 0 -> xyz=0 -0.0635 -0.0762 rpy=1.570796326794896558 0 0
- joint rev_x: origin xyz=0.0076185226336969169569 0.016022870570001249146 -0.026352584457783323479 rpy=1.570796326794896558 -0 1.570796326794896558 -> xyz=0.0076185226336969169569 0.016022870570001249146 -0.026352584457783323479 rpy=1.570796326794896558 0 1.570796326794896558
- joint rev_y: origin xyz=0.10286852263369694604 0.092222870570001252988 -0.026352584457783316541 rpy=-1.570796326794896558 -0 0 -> xyz=0.10286852263369694604 0.092222870570001252988 -0.026352584457783316541 rpy=-1.570796326794896558 0 0

Commit message: more numerical modifications

File: robot.urdf (robot description, URDF)
Before this commit: robot onshape, 4 links, 3 joints
Joints:
- joint cyl_z: origin xyz=0 -0.0635 -0.0762 rpy=1.570796326794896558 0 0 -> xyz=0.0 -0.0635 -0.0762 rpy=1.570796326794896558 0.0 0.0
- joint rev_x: origin xyz=0.0076185226336969169569 0.016022870570001249146 -0.026352584457783323479 rpy=1.570796326794896558 0 1.570796326794896558 -> xyz=0.0076185226336969169569 0.016022870570001249146 -0.026352584457783323479 rpy=1.570796326794896558 0.0 1.570796326794896558
- joint rev_y: origin xyz=0.10286852263369694604 0.092222870570001252988 -0.026352584457783316541 rpy=-1.570796326794896558 0 0 -> xyz=0.10286852263369694604 0.092222870570001252988 -0.026352584457783316541 rpy=-1.570796326794896558 0.0 0.0
