Commit message: first operational test

File: description/robot_core.xacro (robot description, xacro)
@@ -4,10 +4,10 @@
     <link name="base_link">
     </link>
-    <!-- BODY LINK -->
     <joint name="body_joint" type="fixed">
         <parent link="base_link" />
-        <child link="body" />
-        <origin xyz="0.0 0.0 0.0" rpy="0 0 1.57079632679489" />
+        <child link="coupler" />
+        <origin xyz="0.0 0.0 1.0" rpy="0 0 1.57079632679489" />
     </joint>
+    <!-- BODY LINK -->
     <link name="body">
         <visual>
@@ -15,5 +15,5 @@
                 rpy="-1.570796326794896558 -1.570796326794896558 0" />
             <geometry>
-                <mesh filename="package:///body.stl" />
+                <mesh filename="package://hopper/stl/body.stl" />
             </geometry>
             <material name="body_material">
@@ -26,5 +26,5 @@
                 rpy="-1.570796326794896558 -1.570796326794896558 0" />
             <geometry>
-                <mesh filename="package:///body.stl" />
+                <mesh filename="package://hopper/stl/body.stl" />
             </geometry>
         </collision>
@@ -44,5 +44,5 @@
                 rpy="0.0 0.0 0.0" />
             <geometry>
-                <mesh filename="package:///coupler.stl" />
+                <mesh filename="package://hopper/stl/coupler.stl" />
             </geometry>
             <material name="coupler_material">
@@ -55,5 +55,5 @@
                 rpy="0.0 0.0 0.0" />
             <geometry>
-                <mesh filename="package:///coupler.stl" />
+                <mesh filename="package://hopper/stl/coupler.stl" />
             </geometry>
         </collision>
@@ -72,5 +72,5 @@
                 rpy="-1.570796326794896558 0.0 0.0" />
             <geometry>
-                <mesh filename="package:///sleeve.stl" />
+                <mesh filename="package://hopper/stl/sleeve.stl" />
             </geometry>
             <material name="sleeve_material">
@@ -83,5 +83,5 @@
                 rpy="-1.570796326794896558 0.0 0.0" />
             <geometry>
-                <mesh filename="package:///sleeve.stl" />
+                <mesh filename="package://hopper/stl/sleeve.stl" />
             </geometry>
         </collision>
@@ -101,5 +101,5 @@
             <origin xyz="0.0 0.0 -0.9144" rpy="0.0 0.0 0.0" />
             <geometry>
-                <mesh filename="package:///pogo.stl" />
+                <mesh filename="package://hopper/stl/pogo.stl" />
             </geometry>
             <material name="pogo_material">
@@ -111,5 +111,5 @@
             <origin xyz="0.0 0.0 -0.9144" rpy="0.0 0.0 0.0" />
             <geometry>
-                <mesh filename="package:///pogo.stl" />
+                <mesh filename="package://hopper/stl/pogo.stl" />
             </geometry>
         </collision>
@@ -124,6 +124,6 @@
     </link>
     <joint name="rev_x" type="revolute">
-        <origin xyz="0.0076185226336969169569 0.016022870570001249146 -0.026352584457783323479"
-            rpy="1.570796326794896558 0.0 1.570796326794896558" />
+        <!-- <origin xyz="0.076185226336969169569 0.016022870570001249146 -0.026352584457783323479"
+            rpy="1.570796326794896558 0.0 1.570796326794896558" /> -->
         <parent link="coupler" />
         <child link="body" />

Commit message: update mesh uri's

File: description/robot_core.xacro (robot description, xacro)
@@ -15,5 +15,5 @@
                 rpy="-1.570796326794896558 -1.570796326794896558 0" />
             <geometry>
-                <mesh filename="package://hopper/stl/body.stl" />
+                <mesh filename="package://hopper-description/stl/body.stl" />
             </geometry>
             <material name="body_material">
@@ -26,5 +26,5 @@
                 rpy="-1.570796326794896558 -1.570796326794896558 0" />
             <geometry>
-                <mesh filename="package://hopper/stl/body.stl" />
+                <mesh filename="package://hopper-description/stl/body.stl" />
             </geometry>
         </collision>
@@ -44,5 +44,5 @@
                 rpy="0.0 0.0 0.0" />
             <geometry>
-                <mesh filename="package://hopper/stl/coupler.stl" />
+                <mesh filename="package://hopper-description/stl/coupler.stl" />
             </geometry>
             <material name="coupler_material">
@@ -55,5 +55,5 @@
                 rpy="0.0 0.0 0.0" />
             <geometry>
-                <mesh filename="package://hopper/stl/coupler.stl" />
+                <mesh filename="package://hopper-description/stl/coupler.stl" />
             </geometry>
         </collision>
@@ -72,5 +72,5 @@
                 rpy="-1.570796326794896558 0.0 0.0" />
             <geometry>
-                <mesh filename="package://hopper/stl/sleeve.stl" />
+                <mesh filename="package://hopper-description/stl/sleeve.stl" />
             </geometry>
             <material name="sleeve_material">
@@ -83,5 +83,5 @@
                 rpy="-1.570796326794896558 0.0 0.0" />
             <geometry>
-                <mesh filename="package://hopper/stl/sleeve.stl" />
+                <mesh filename="package://hopper-description/stl/sleeve.stl" />
             </geometry>
         </collision>
@@ -101,5 +101,5 @@
             <origin xyz="0.0 0.0 -0.9144" rpy="0.0 0.0 0.0" />
             <geometry>
-                <mesh filename="package://hopper/stl/pogo.stl" />
+                <mesh filename="package://hopper-description/stl/pogo.stl" />
             </geometry>
             <material name="pogo_material">
@@ -111,5 +111,5 @@
             <origin xyz="0.0 0.0 -0.9144" rpy="0.0 0.0 0.0" />
             <geometry>
-                <mesh filename="package://hopper/stl/pogo.stl" />
+                <mesh filename="package://hopper-description/stl/pogo.stl" />
             </geometry>
         </collision>

Commit message: update robot_core.xacro

File: description/robot_core.xacro (robot description, xacro)
@@ -12,6 +12,5 @@
     <link name="body">
         <visual>
-            <origin xyz="0.0 0.0 0.0"
-                rpy="-1.570796326794896558 -1.570796326794896558 0" />
+            <origin xyz="0 0 0" rpy="0 0 0" />
             <geometry>
                 <mesh filename="package:///body.stl" />
@@ -23,6 +22,5 @@
         </visual>
         <collision>
-            <origin xyz="0.0 -0.1016 0.09525"
-                rpy="-1.570796326794896558 -1.570796326794896558 0" />
+            <origin xyz="0 0 0" rpy="0 0 0" />
             <geometry>
                 <mesh filename="package:///body.stl" />
@@ -30,10 +28,9 @@
         </collision>
         <inertial>
-            <origin xyz="0.00094664124949074362168 0.0019566509168293666487 0.095175461021671584061"
-                rpy="0.0 0.0 0.0" />
+            <origin xyz="-7.4538978328428899403e-05 0.00094664124949074969322 0.10355665091682933476" rpy="0 0 0" />
             <mass value="71.513617955613540289" />
-            <inertia ixx="2.7695768268605731599" ixy="-0.012891515253177195446"
-                ixz="-5.0461204235767260229e-06" iyy="4.9414740165599875255"
-                iyz="-1.0430029495049975829e-05" izz="2.7059577965441983238" />
+            <inertia ixx="2.7059577965441987679" ixy="-5.0461204235837386087e-06"
+                ixz="-1.0430029495029113408e-05" iyy="2.7695768268605731599"
+                iyz="-0.01289151525317717116" izz="4.9414740165599875255" />
         </inertial>
     </link>
@@ -41,6 +38,6 @@
     <link name="coupler">
         <visual>
-            <origin xyz="0.0076185226336969169569 0.01602287057000122833 -0.026352584457783326949"
-                rpy="0.0 0.0 0.0" />
+            <origin xyz="-2.0816681711721685133e-17 0 0.0063499999999999945377"
+                rpy="1.570796326794896558 1.570796326794896558 0" />
             <geometry>
                 <mesh filename="package:///coupler.stl" />
@@ -52,6 +49,6 @@
         </visual>
         <collision>
-            <origin xyz="0.0076185226336969169569 0.01602287057000122833 -0.026352584457783326949"
-                rpy="0.0 0.0 0.0" />
+            <origin xyz="-2.0816681711721685133e-17 0 0.0063499999999999945377"
+                rpy="1.570796326794896558 1.570796326794896558 0" />
             <geometry>
                 <mesh filename="package:///coupler.stl" />
@@ -59,9 +56,10 @@
         </collision>
         <inertial>
-            <origin xyz="0.059457331089903711629 0.04473059794826811375 -0.026352584457783306132"
-                rpy="0.0 0.0 0.0" />
+            <origin
+                xyz="0.028707727378266875012 -1.6124666532645141538e-17 -0.045488808456206786257"
+                rpy="0 0 0" />
             <mass value="0.52500488643203435668" />
-            <inertia ixx="0.0017154388189821222557" ixy="-0.0007995744266173912063" ixz="0.0"
-                iyy="0.0026160173506496889675" iyz="0.0" izz="0.0029912187796853682668" />
+            <inertia ixx="0.0026160173506496889675" ixy="0" ixz="0.00079957442661739131472"
+                iyy="0.0029912187796853669658" iyz="0" izz="0.0017154388189821222557" />
         </inertial>
     </link>
@@ -69,6 +67,6 @@
     <link name="sleeve">
         <visual>
-            <origin xyz="0.0 0.0 -0.0762"
-                rpy="-1.570796326794896558 0.0 0.0" />
+            <origin xyz="-3.0814879110195773649e-33 0 -0.076200000000000003841"
+                rpy="-1.570796326794896558 -0 0" />
             <geometry>
                 <mesh filename="package:///sleeve.stl" />
@@ -80,6 +78,6 @@
         </visual>
         <collision>
-            <origin xyz="0.0 0.0 -0.0762"
-                rpy="-1.570796326794896558 0.0 0.0" />
+            <origin xyz="-3.0814879110195773649e-33 0 -0.076200000000000003841"
+                rpy="-1.570796326794896558 -0 0" />
             <geometry>
                 <mesh filename="package:///sleeve.stl" />
@@ -88,6 +86,6 @@
         <inertial>
             <origin
-                xyz="0.0 0.0 -0.060135671624197417628"
-                rpy="0.0 0.0 0.0" />
+                xyz="-1.278090274607719524e-08 7.890502699878677037e-09 -0.060135671624197403751"
+                rpy="0 0 0" />
             <mass value="0.4777148575757113047" />
             <inertia ixx="0.00098751957755369027328" ixy="1.8087162374182167824e-10"
@@ -99,5 +97,5 @@
     <link name="pogo">
         <visual>
-            <origin xyz="0.0 0.0 -0.9144" rpy="0.0 0.0 0.0" />
+            <origin xyz="0 -1.1664760761878542743e-18 -0.91440000000000010161" rpy="0 -0 0" />
             <geometry>
                 <mesh filename="package:///pogo.stl" />
@@ -109,5 +107,5 @@
         </visual>
         <collision>
-            <origin xyz="0.0 0.0 -0.9144" rpy="0.0 0.0 0.0" />
+            <origin xyz="0 -1.1664760761878542743e-18 -0.91440000000000010161" rpy="0 -0 0" />
             <geometry>
                 <mesh filename="package:///pogo.stl" />
@@ -116,6 +114,6 @@
         <inertial>
             <origin
-                xyz="0.0 0.0 -0.45403610139860128836"
-                rpy="0.0 0.0 0.0" />
+                xyz="4.3194544932116136525e-19 -1.9259299443872358531e-34 -0.45403610139860128836"
+                rpy="0 0 0" />
             <mass value="1.0890939243757413735" />
             <inertia ixx="0.074944292622089278555" ixy="0.0" ixz="0.0" iyy="0.074944292622089278555"
@@ -123,16 +121,7 @@
         </inertial>
     </link>
-    <joint name="rev_x" type="revolute">
-        <origin xyz="0.0076185226336969169569 0.016022870570001249146 -0.026352584457783323479"
-            rpy="1.570796326794896558 0.0 1.570796326794896558" />
-        <parent link="coupler" />
-        <child link="body" />
-        <axis xyz="0 0 1" />
-        <limit effort="1.5" velocity="22" />
-        <joint_properties friction="0.0" />
-    </joint>
-    <joint name="cyl_z" type="prismatic">
-        <origin xyz="0.0 -0.0635 -0.0762"
-            rpy="1.570796326794896558 0.0 0.0" />
+    <joint name="pri_z" type="prismatic">
+        <origin xyz="3.4694469519536141888e-18 -0.063500000000000070277 -0.076200000000000003841"
+            rpy="1.570796326794896558 -0 0" />
         <parent link="sleeve" />
         <child link="pogo" />
@@ -142,6 +131,6 @@
     </joint>
     <joint name="rev_y" type="revolute">
-        <origin xyz="0.10286852263369694604 0.092222870570001252988 -0.026352584457783316541"
-            rpy="-1.570796326794896558 0.0 0.0" />
+        <origin xyz="0.076199999999999989964 -1.3877787807814456755e-17 -0.088900000000000006795"
+            rpy="-0 1.570796326794896558 0" />
         <parent link="coupler" />
         <child link="sleeve" />
@@ -150,3 +139,12 @@
         <joint_properties friction="0.0" />
     </joint>
+    <joint name="rev_x" type="revolute">
+        <origin xyz="-0.088900000000000020672 -5.2041704279304212832e-18 0.10159999999999994036"
+            rpy="-1.570796326794896558 -0 1.57079632679489678" />
+        <parent link="body" />
+        <child link="coupler" />
+        <axis xyz="0 0 1" />
+        <limit effort="1.5" velocity="22" />
+        <joint_properties friction="0.0" />
+    </joint>
 </robot>
